Commit message: manual merge up to commit cff9fe91fc299433f3e091eded51b5084f930410

File: robots/gen3.xacro (robot description, xacro)
@@ -3,7 +3,10 @@
     <!-- Arguments -->
     <xacro:arg name="arm" default="gen3" />
+    <xacro:arg name="dof" default="7" />
+    <xacro:arg name="vision" default="true" />
     <xacro:arg name="gripper" default="" />
     <xacro:arg name="sim" default="false" />
+    <xacro:arg name="prefix" default="" />
     <xacro:include filename="$(find kortex_description)/robots/kortex_robot.xacro" />
-    <xacro:load_robot arm="$(arg arm)" gripper="$(arg gripper)" sim="$(arg sim)" />
+    <xacro:load_robot arm="$(arg arm)" gripper="$(arg gripper)" dof="$(arg dof)" vision="$(arg vision)" sim="$(arg sim)" prefix="$(arg prefix)" />
 </robot>

File: robots/gen3_robotiq_2f_85.xacro (robot description, xacro)
@@ -3,7 +3,10 @@
     <!-- Arguments -->
     <xacro:arg name="arm" default="gen3" />
+    <xacro:arg name="dof" default="7" />
+    <xacro:arg name="vision" default="true" />
     <xacro:arg name="gripper" default="robotiq_2f_85" />
     <xacro:arg name="sim" default="false" />
+    <xacro:arg name="prefix" default="" />
     <xacro:include filename="$(find kortex_description)/robots/kortex_robot.xacro" />
-    <xacro:load_robot arm="$(arg arm)" gripper="$(arg gripper)" sim="$(arg sim)"/>
+    <xacro:load_robot arm="$(arg arm)" gripper="$(arg gripper)" dof="$(arg dof)" vision="$(arg vision)" sim="$(arg sim)" prefix="$(arg prefix)" />
 </robot>

File: robots/kortex_robot.xacro (robot description, xacro)
@@ -1,25 +1,21 @@
 <?xml version="1.0"?>
 <robot xmlns:xacro="http://ros.org/wiki/xacro">
-    <xacro:macro name="load_robot" params="arm gripper sim">
-        <!-- Arguments -->
-        <xacro:property name="arm" value="$(arg arm)" />
-        <xacro:property name="gripper" default="$(arg gripper)" />
-        <xacro:property name="sim" default="$(arg sim)" />
+    <xacro:macro name="load_robot" params="arm gripper dof vision sim prefix">
         <!-- Files to include -->
-        <xacro:include filename="$(find kortex_description)/arms/$(arg arm)/urdf/$(arg arm)_macro.xacro" />
+        <xacro:include filename="$(find kortex_description)/arms/${arm}/${dof}dof/urdf/${arm}_macro.xacro" />
         <xacro:unless value="${not gripper}">
-            <xacro:include filename="$(find kortex_description)/grippers/$(arg gripper)/urdf/$(arg gripper)_macro.xacro" />
+            <xacro:include filename="$(find kortex_description)/grippers/${gripper}/urdf/${gripper}_macro.xacro" />
         </xacro:unless>
-        <xacro:if value="$(arg sim)">
+        <xacro:if value="${sim}">
             <!-- Arm transmission elements-->
-            <xacro:include filename="$(find kortex_description)/arms/$(arg arm)/urdf/$(arg arm)_transmission_macro.xacro" />
+            <xacro:include filename="$(find kortex_description)/arms/${arm}/${dof}dof/urdf/${arm}_transmission_macro.xacro" />
             <!-- Gripper transmission elements if there is a gripper-->
             <xacro:unless value="${not gripper}">
-                <xacro:include filename="$(find kortex_description)/grippers/$(arg gripper)/urdf/$(arg gripper)_transmission_macro.xacro" />
+                <xacro:include filename="$(find kortex_description)/grippers/${gripper}/urdf/${gripper}_transmission_macro.xacro" />
             </xacro:unless>
         </xacro:if>
         <!-- Run the macros -->
         <!-- For gazebo-->
-        <xacro:if value="$(arg sim)">
+        <xacro:if value="${sim}">
             <link name="world" />
             <joint name="world_to_root" type="fixed">
@@ -30,16 +26,17 @@
         </xacro:if>
         <!-- Load the arm -->
-        <xacro:load_arm parent="">
+        <xacro:load_arm parent="" dof="${dof}" vision="${vision}" prefix="${prefix}">
             <origin xyz="0 0 0" rpy="0 0 0"/>
         </xacro:load_arm>
         <!-- Load the gripper -->
         <xacro:unless value="${not gripper}">
-            <xacro:load_gripper parent="${last_arm_link}"/> <!-- last_arm_link is defined in "$(find kortex_description)/arms/$(arg arm)/urdf/$(arg arm)_macro.xacro" -->
+            <!-- last_arm_link is defined in "$(find kortex_description)/arms/${arm}/urdf/${arm}_macro.xacro" -->
+            <xacro:load_gripper parent="${prefix}${last_arm_link}"  prefix="${prefix}"/>
         </xacro:unless>
         <!-- Load the Gazebo transmissions and gazebo_ros_control plugin -->
-        <xacro:if value="$(arg sim)">
-            <xacro:load_gazebo_arm_transmissions/>
+        <xacro:if value="${sim}">
+            <xacro:load_gazebo_arm_transmissions prefix="${prefix}"/>
             <xacro:unless value="${not gripper}">
-                <xacro:load_gazebo_gripper_transmissions/>
+                <xacro:load_gazebo_gripper_transmissions prefix="${prefix}"/>
             </xacro:unless>
             <gazebo>
